Commit message: Mon Jul  1 15:18:07 CST 2019 add idealfish_velocity_controller

File: idealfish_description/urdf/base.gazebo.xacro (robot description, xacro)
@@ -1,5 +1,5 @@
 <?xml version="1.0" ?>
 <robot name="idealfish" xmlns:xacro="https://www.ros.org/wiki/xacro" >
-  <gazebo reference="link_chassis">
+  <gazebo reference="base_link">
     <material>Gazebo/Orange</material>
   </gazebo>
@@ -22,5 +22,5 @@
       <odometryTopic>odom</odometryTopic>
       <odometryFrame>odom</odometryFrame>
-      <robotBaseFrame>link_chassis</robotBaseFrame>
+      <robotBaseFrame>base_link</robotBaseFrame>
     </plugin>
   </gazebo-->

File: idealfish_description/urdf/base.urdf.xacro (robot description, xacro)
@@ -5,5 +5,5 @@
   <xacro:include filename="$(find idealfish_description)/urdf/wheel.macro.xacro"/>
   <xacro:include filename="$(find idealfish_description)/urdf/base.transmission.xacro"/>
-  <link name="link_chassis">
+  <link name="base_link">
     <!-- pose and inertial -->
     <pose>0 0 0.1 0 0 0</pose>

File: idealfish_description/urdf/wheel.macro.xacro (robot description, xacro)
@@ -26,5 +26,5 @@
         <origin rpy="0 0 0" xyz="${origin_xyz}"/>
         <child link="${child}"/>
-        <parent link="link_chassis"/>
+        <parent link="base_link"/>
         <axis rpy="0 0 0" xyz="0 1 0"/>
         <limit effort="10000" velocity="1000"/>

Commit message: Mon Jul  1 18:42:10 CST 2019 real world size model, good in rviz, drift in gazebo

File: idealfish_description/urdf/base.gazebo.xacro (robot description, xacro)
@@ -6,7 +6,17 @@
   <gazebo reference="link_left_wheel">
     <material>Gazebo/Blue</material>
+    <mu1 value="1.0"/>
+    <mu2 value="1.0"/>
+    <kp value="10000000.0" />
+    <kd value="1.0" />
+    <fdir1 value="1 0 0"/>
   </gazebo>
   <gazebo reference="link_right_wheel">
     <material>Gazebo/Blue</material>
+    <mu1 value="1.0"/>
+    <mu2 value="1.0"/>
+    <kp value="10000000.0" />
+    <kd value="1.0" />
+    <fdir1 value="1 0 0"/>
   </gazebo>
   <!--gazebo>

File: idealfish_description/urdf/base.urdf.xacro (robot description, xacro)
@@ -5,29 +5,31 @@
   <xacro:include filename="$(find idealfish_description)/urdf/wheel.macro.xacro"/>
   <xacro:include filename="$(find idealfish_description)/urdf/base.transmission.xacro"/>
+  <xacro:property name="M_PI" value="3.14159"/>
   <link name="base_link">
     <!-- pose and inertial -->
     <pose>0 0 0.1 0 0 0</pose>
+    <!-- base -->
     <inertial>
       <mass value="5"/>
-      <origin rpy="0 0 0" xyz="0 0 0.1"/>
-      <inertia ixx="0.0395416666667" ixy="0" ixz="0" iyy="0.106208333333" iyz="0" izz="0.106208333333"/>
+      <origin rpy="0 0 0" xyz="-0.09 0 0"/> <!--0.36/2 - 0.09-->
+      <inertia ixx="0.0560416666667" ixy="0" ixz="0" iyy="0.0395416666667" iyz="0" izz="0.0915"/>
     </inertial>
-    <collision name="collision_chassis">
+    <collision name="collision_base_link">
       <geometry>
-        <box size="0.5 0.3 0.07"/>
+        <box size="0.36 0.3 0.08"/>
       </geometry>
     </collision>
     <visual>
-      <origin rpy="0 0 0" xyz="0 0 0"/>
+      <origin rpy="0 0 0" xyz="-0.09 0 0"/>
       <geometry>
-        <box size="0.5 0.3 0.07"/>
+        <box size="0.36 0.3 0.08"/>
       </geometry>
       <material name="blue"/>
     </visual>
-    <!-- caster front -->
+    <!-- caster back -->
     <collision name="caster_front_collision">
-      <origin rpy=" 0 0 0" xyz="0.35 0 -0.05"/>
+      <origin rpy=" 0 0 0" xyz="-0.27 0 -0.07"/><!--0.36-0.09=0.27-->
       <geometry>
-        <sphere radius="0.05"/>
+        <sphere radius="0.03"/>
       </geometry>
       <surface>
@@ -43,7 +45,7 @@
     </collision>
     <visual name="caster_front_visual">
-      <origin rpy=" 0 0 0" xyz="0.2 0 -0.05"/>
+      <origin rpy=" 0 0 0" xyz="-0.27 0 -0.07"/><!--0.36-0.09=0.27-->
       <geometry>
-        <sphere radius="0.05"/>
+        <sphere radius="0.03"/>
       </geometry>
     </visual>
@@ -53,6 +55,6 @@
   <xacro:link_wheel name="link_left_wheel"/>
   <!-- Create wheel right, left joint -->
-  <xacro:joint_wheel name="joint_right_wheel" child="link_right_wheel" origin_xyz="-0.05 0.15 0"/>
-  <xacro:joint_wheel name="joint_left_wheel" child="link_left_wheel" origin_xyz="-0.05 -0.15 0"/>
+  <xacro:joint_wheel name="joint_right_wheel" child="link_right_wheel" origin_xyz="-0.0 0.17 0"/><!--width = 0.3/2+0.005+0.03/2-->
+  <xacro:joint_wheel name="joint_left_wheel" child="link_left_wheel" origin_xyz="-0.0 -0.17 0"/><!--0.3/2+0.005+0.03/2-->
   <!-- Create wheel right, left transmission -->
   <xacro:right_wheel_trans/>

File: idealfish_description/urdf/wheel.macro.xacro (robot description, xacro)
@@ -4,18 +4,18 @@
         <link name="${name}">
             <inertial>
-              <mass value="0.2"/>
-              <origin rpy="0 1.5707 1.5707" xyz="0 0 0"/>
-              <inertia ixx="0.000526666666667" ixy="0" ixz="0" iyy="0.000526666666667" iyz="0" izz="0.001"/>
+              <mass value="2.5"/>
+              <origin rpy="0 ${M_PI/2} ${M_PI/2}" xyz="0 0 0"/>
+              <inertia  ixx="0.02467" ixy="0" ixz="0" iyy="0.04411" iyz="0" izz="0.02467" />
             </inertial>
             <collision name="link_right_wheel_collision">
-              <origin rpy="0 1.5707 1.5707" xyz="0 0 0"/>
+              <origin rpy="0 ${M_PI/2} ${M_PI/2}" xyz="0 0 0"/>
               <geometry>
-                <cylinder length="0.04" radius="0.1"/>
+                <cylinder length="0.03" radius="0.1"/>
               </geometry>
             </collision>
             <visual name="${name}_visual">
-              <origin rpy="0 1.5707 1.5707" xyz="0 0 0"/>
+              <origin rpy="0 ${M_PI/2} ${M_PI/2}" xyz="0 0 0"/>
               <geometry>
-                <cylinder length="0.04" radius="0.1"/>
+                <cylinder length="0.03" radius="0.1"/>
               </geometry>
             </visual>

Commit message: find the bug is at wheel

File: idealfish_description/urdf/base.gazebo.xacro (robot description, xacro)
@@ -2,4 +2,7 @@
 <robot name="idealfish" xmlns:xacro="https://www.ros.org/wiki/xacro" >
   <gazebo reference="base_link">
+    <material>Gazebo/Orange</material>
+  </gazebo>
+  <gazebo reference="body_link">
     <material>Gazebo/Orange</material>
   </gazebo>

File: idealfish_description/urdf/base.urdf.xacro (robot description, xacro)
@@ -7,11 +7,23 @@
   <xacro:property name="M_PI" value="3.14159"/>
   <link name="base_link">
-    <!-- pose and inertial -->
-    <pose>0 0 0.1 0 0 0</pose>
+    <visual>
+      <origin xyz="0 0 0" rpy="0 0 0"/>
+      <geometry>
+        <box size="0.01 0.01 0.01" />
+      </geometry>
+      <material name="White" />
+    </visual>
+  </link>
+  <joint name="base_link_joint" type="fixed">
+    <origin xyz="-0.09 0 0" rpy="0 0 0"/>
+    <parent link="base_link"/>
+    <child link="body_link" />
+  </joint>
+  <link name="body_link">
     <!-- base -->
     <inertial>
-      <mass value="5"/>
-      <origin rpy="0 0 0" xyz="-0.09 0 0"/> <!--0.36/2 - 0.09-->
-      <inertia ixx="0.0560416666667" ixy="0" ixz="0" iyy="0.0395416666667" iyz="0" izz="0.0915"/>
+      <mass value="10"/>
+      <origin rpy="0 0 0" xyz="0 0 0"/> <!--0.36/2 - 0.09-->
+      <inertia ixx="0.0803333333333" ixy="0" ixz="0" iyy="0.11333333333" iyz="0" izz="0.183"/>
     </inertial>
     <collision name="collision_base_link">
@@ -21,5 +33,5 @@
     </collision>
     <visual>
-      <origin rpy="0 0 0" xyz="-0.09 0 0"/>
+      <origin rpy="0 0 0" xyz="0 0 0"/>
       <geometry>
         <box size="0.36 0.3 0.08"/>
@@ -29,5 +41,5 @@
     <!-- caster back -->
     <collision name="caster_front_collision">
-      <origin rpy=" 0 0 0" xyz="-0.27 0 -0.07"/><!--0.36-0.09=0.27-->
+      <origin rpy=" 0 0 0" xyz="-0.18 0 -0.07"/><!--0.08/2+0.03-->
       <geometry>
         <sphere radius="0.03"/>
@@ -45,5 +57,5 @@
     </collision>
     <visual name="caster_front_visual">
-      <origin rpy=" 0 0 0" xyz="-0.27 0 -0.07"/><!--0.36-0.09=0.27-->
+      <origin rpy=" 0 0 0" xyz="-0.18 0 -0.07"/><!--0.36-0.09=0.27-->
       <geometry>
         <sphere radius="0.03"/>
